File: implant_hardware_sch/implant_hardware_sch.kicad_sch (KiCad schematic)
At the start: 24 parts, among them IC1 XCL101A301ER-G, IC2 MUX, IC3 CYBLE-214015-01, J1 Conn_01x02, U1 MIC5365-1.8YMT-TZ, U2 MIC5365-1.8YMT-TZ, U3 MIC5365-2.0YMT-TZ, U4 MIC5365-2.5YMT-TZ, Y1 2.5MHz Oscillator

Commit message: Updated KiCad schematic
Parts:
- IC1: value XCL101A301ER-G -> DC-DC
- IC3: value CYBLE-214015-01 -> MCU
- J1: value Conn_01x02 -> Battery
- U1, U2: value MIC5365-1.8YMT-TZ -> 1.8V LDO
- U3: value MIC5365-2.0YMT-TZ -> 2.0V LDO
- U4: value MIC5365-2.5YMT-TZ -> 2.5V LDO
Connections:
- net 1.8V: now also FB4.1, FB5.2, Y1.4 (VDD); no longer FB1.1, FB2.1
- net GND: now also Y1.2 (GND)
- net at FB5.1: no longer IC3.7 (VDD)
- net at C8.1, U2.1 (VOUT): now also FB1.1, FB3.1; no longer FB4.1, FB5.2
- net at C9.1, U3.1 (VOUT): now also FB2.2; no longer FB3.1
- net CLK_2P5M: now reaches Y1.3 (OUT)
- net EN: now reaches IC3.12 (P1.2)
- net EN: now also IC2.1 (EN)
- net at FB3.2: now also IC3.20 (VDDA); no longer IC3.13 (VDDR)
- net D_ADC_strobe: now reaches IC3.16 (P3.0)
- net D_APT_reset: now reaches IC3.18 (P2.2)
- net D_APT_reset: now also IC3.19 (P2.3)
- net at FB4.2: no longer IC3.20 (VDDA)
- net CLK100kHz: now reaches IC3.21 (P3.4)
- net CLK10kHz: now reaches IC3.22 (P3.1)
- net SCANDACSIN: now reaches IC3.23 (P3.7)
- net SCANDACEN: now reaches IC3.24 (P3.5)
- net SCANDACSOUT: now reaches IC3.25 (P3.3)
- net SCANMAINSIN: now reaches IC3.27 (P3.2)
- net SCANMAINEN: now reaches IC3.28 (P3.6)
- net SCANMAINSCLK: now reaches IC3.29 (XRES)
- net SCANMAINSOUT: now reaches IC3.30 (P2.4)
- net D_ADC_SIOC: now reaches IC3.8 (P1.4)
- net D_ADC_SIOD: now reaches IC3.9 (P0.4)
- net 2.5V: now reaches U4.5
- net at FB1.2: now also IC3.7 (VDD)
- new net: FB2.1, IC3.13 (VDDR)
Other:
- title: (none) -> Implant Hardware
- moved on the sheet: C1, C10, C2, C3, C4, C5, C6, C7, C8, C9, FB1, FB2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
